File: pcb/ndice.brd (EAGLE design)
At the start: 23.6 x 26 mm, 19 parts, among them U1 ATTINY1614-SSNR

Commit message: updated eagle brd file
Routing:
- net N$1: track 4.91 -> 5.45 mm
Changed lines of the file:
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@@
 <?xml version="1.0" encoding="utf-8"?>
 <!DOCTYPE eagle SYSTEM "eagle.dtd">
-<eagle version="9.1.0">
+<eagle version="9.3.0">
 <drawing>
 <settings>
@@
 <layers>
 <layer number="1" name="Top" color="4" fill="1" visible="yes" active="yes"/>
+<layer number="2" name="Route2" color="1" fill="3" visible="no" active="no"/>
+<layer number="3" name="Route3" color="4" fill="3" visible="no" active="no"/>
+<layer number="4" name="Route4" color="1" fill="4" visible="no" active="no"/>
+<layer number="5" name="Route5" color="4" fill="4" visible="no" active="no"/>
+<layer number="6" name="Route6" color="1" fill="8" visible="no" active="no"/>
+<layer number="7" name="Route7" color="4" fill="8" visible="no" active="no"/>
+<layer number="8" name="Route8" color="1" fill="2" visible="no" active="no"/>
+<layer number="9" name="Route9" color="4" fill="2" visible="no" active="no"/>
+<layer number="10" name="Route10" color="1" fill="7" visible="no" active="no"/>
+<layer number="11" name="Route11" color="4" fill="7" visible="no" active="no"/>
+<layer number="12" name="Route12" color="1" fill="5" visible="no" active="no"/>
+<layer number="13" name="Route13" color="4" fill="5" visible="no" active="no"/>
+<layer number="14" name="Route14" color="1" fill="6" visible="no" active="no"/>
+<layer number="15" name="Route15" color="4" fill="6" visible="no" active="no"/>
 <layer number="16" name="Bottom" color="1" fill="1" visible="yes" active="yes"/>
 <layer number="17" name="Pads" color="2" fill="1" visible="yes" active="yes"/>
@@
 </class>
 </classes>
-<designrules name="dirt_cheap_dirty_boards.v1.1">
-<description language="de">&lt;b&gt;Dirty Cheap Dirty Board Design Rules&lt;/b&gt;
-&lt;br&gt;
-&lt;br&gt;Min width/Spacing: 6/6mil
-&lt;br&gt;Min diameter of finished hole 12mil</description>
-<description language="en">&lt;b&gt;Dirty Cheap Dirty Board Design Rules&lt;/b&gt;
-&lt;br&gt;
-&lt;br&gt;Min width/Spacing: 6/6mil
-&lt;br&gt;Min diameter of finished hole 12mil</description>
-<description language="zh">&lt;b&gt;Dirty Cheap Dirty Board Design Rules&lt;/b&gt;
-&lt;br&gt;
-&lt;br&gt;Min width/Spacing: 6/6mil
-&lt;br&gt;Min diameter of finished hole 12mil</description>
+<designrules name="SeeedStudio_2layer_DRU_no_angle_20140221">
+<description language="de">&lt;b&gt;EAGLE Design Rules&lt;/b&gt;
+&lt;p&gt;
+Die Standard-Design-Rules sind so gewählt, dass sie für
+die meisten Anwendungen passen. Sollte ihre Platine
+besondere Anforderungen haben, treffen Sie die erforderlichen
+Einstellungen hier und speichern die Design Rules unter
+einem neuen Namen ab.</description>
+<description language="en">&lt;b&gt;EAGLE Design Rules&lt;/b&gt;
+&lt;p&gt;
+The default Design Rules have been set to cover
+a wide range of applications. Your particular design
+may have different requirements, so please make the
+necessary adjustments and save your customized
+design rules under a new name.</description>
+<description language="zh">&lt;b&gt;Seeed Studio EAGLE Design Rules&lt;/b&gt;
+</description>
 <param name="layerSetup" value="(1*16)"/>
 <param name="mtCopper" value="0.035mm 0.0175mm 0.035mm 0.035mm 0.035mm 0.035mm 0.035mm 0.035mm 0.035mm 0.035mm 0.035mm 0.035mm 0.035mm 0.035mm 0.0175mm 0.035mm"/>
@@
 <param name="mlMinCreamFrame" value="0mil"/>
 <param name="mlMaxCreamFrame" value="0mil"/>
-<param name="mlViaStopLimit" value="25mil"/>
+<param name="mlViaStopLimit" value="100mil"/>
 <param name="srRoundness" value="0"/>
 <param name="srMinRoundness" value="0mil"/>
@@
 <vertex x="2.54" y="1.27"/>
 </polygon>
-<wire x1="13.250803125" y1="22.70834375" x2="13.250803125" y2="21.480803125" width="0.1524" layer="1"/>
+<wire x1="12.8541875" y1="23.08690625" x2="13.250803125" y2="21.480803125" width="0.1524" layer="1"/>
 <wire x1="13.250803125" y1="21.480803125" x2="12.74" y2="20.97" width="0.1524" layer="1"/>
 </signal>
@@
 <wire x1="17.78" y1="20.93" x2="17.78" y2="17.78" width="0.1524" layer="16"/>
 <contactref element="U$1" pad="P$2"/>
-<wire x1="20.16834375" y1="19.76919375" x2="18.94080625" y2="19.76919375" width="0.2032" layer="1"/>
+<wire x1="20.54690625" y1="20.165809375" x2="18.94080625" y2="19.76919375" width="0.2032" layer="1"/>
 <wire x1="18.94080625" y1="19.76919375" x2="17.74" y2="20.97" width="0.2032" layer="1"/>
-<wire x1="6.096" y1="17.018" x2="7.763178125" y2="18.685178125" width="0.1524" layer="1"/>
-<wire x1="7.763178125" y1="18.685178125" x2="8.425221875" y2="18.685178125" width="0.1524" layer="1"/>
-<wire x1="9.027053125" y1="20.0099625" x2="10.0094875" y2="20.992396875" width="0.1524" layer="1"/>
 <wire x1="15.64700625" y1="19.9874" x2="15.97960625" y2="20.32" width="0.1524" layer="1"/>
-<wire x1="12.33299375" y1="19.9874" x2="15.64700625" y2="19.9874" width="0.1524" layer="1"/>
-<wire x1="8.425221875" y1="18.685178125" x2="9.027053125" y2="19.287009375" width="0.1524" layer="1"/>
-<wire x1="9.027053125" y1="19.287009375" x2="9.027053125" y2="20.0099625" width="0.1524" layer="1"/>
-<wire x1="10.0094875" y1="20.992396875" x2="11.327996875" y2="20.992396875" width="0.1524" layer="1"/>
-<wire x1="11.327996875" y1="20.992396875" x2="12.33299375" y2="19.9874" width="0.1524" layer="1"/>
+<wire x1="13.97" y1="19.9874" x2="15.64700625" y2="19.9874" width="0.1524" layer="1"/>
 <wire x1="17.09" y1="20.32" x2="17.74" y2="20.97" width="0.1524" layer="1"/>
 <wire x1="15.97960625" y1="20.32" x2="17.09" y2="20.32" width="0.1524" layer="1"/>
+<wire x1="6.096" y1="17.018" x2="10.668" y2="17.018" width="0.1524" layer="1"/>
+<wire x1="10.668" y1="17.018" x2="10.922" y2="17.272" width="0.1524" layer="1"/>
+<wire x1="12.6214" y1="19.9874" x2="13.97" y2="19.9874" width="0.1524" layer="1"/>
+<wire x1="10.922" y1="17.272" x2="10.922" y2="18.288" width="0.1524" layer="1"/>
+<wire x1="10.922" y1="18.288" x2="12.6214" y2="19.9874" width="0.1524" layer="1"/>
 </signal>
 <signal name="N$2">
@@
 <wire x1="10.16" y1="16.3331125" x2="10.16" y2="17.78" width="0.1524" layer="16"/>
 <wire x1="10.16" y1="17.78" x2="10.16" y2="19.61754375" width="0.1524" layer="1"/>
-<wire x1="10.16" y1="19.61754375" x2="10.280953125" y2="19.738496875" width="0.1524" layer="1"/>
+<wire x1="10.16" y1="19.61754375" x2="9.837553125" y2="20.181896875" width="0.1524" layer="1"/>
 </signal>
 <signal name="N$3">
@@
 <wire x1="15.24" y1="26.51" x2="15.24" y2="24.13" width="0.2032" layer="1"/>
 <wire x1="15.24" y1="24.13" x2="16.63095625" y2="22.73904375" width="0.2032" layer="1"/>
-<wire x1="16.63095625" y1="22.73904375" x2="17.198496875" y2="22.73904375" width="0.2032" layer="1"/>
+<wire x1="16.63095625" y1="22.73904375" x2="17.641896875" y2="23.18244375" width="0.2032" layer="1"/>
 </signal>
 </signals>
